File: Android_Oscilloscope.kicad_pcb (KiCad board)
At the start: 4 copper layers, 70 x 43 mm, 134 parts, among them J1 BNC, P1 USB_BOOT, P2 FCI_10118193-0001LF, P3 JTAG, U1 LPC4370FET100, U10 USBLC6-2SC6, U11 LM385M3-1.2/NOPB, U12 LM385M3-1.2/NOPB, U13 AT24C02C-XHM-T, U14 MCP4726A0T-E/CH, U2 CPC1017N, U3 AMS1117-3.3, U4 CPC1017N, U5 OPA4354AIPWR, U6 LM2664, U7 74HC4052PW, U8 W25Q80BVSSIG, U9 TC7W53FK, Y1 ABLS-12.000MHZ-B4-T

Commit message: 回路図 DRC pass
Parts:
- removed FID1: Fiducial_C, MyMsc:Fiducial_1mm
- removed FID2: Fiducial_A, MyMsc:Fiducial_1mm
- removed FID3: Fiducial_B, MyMsc:Fiducial_1mm
- added L6: MLP2012H2R2MT0S1, Inductor_SMD:L_0805_2012Metric, F.Cu at (97.3, 129.6)
- added R41: 5.1k 1%, Resistor_SMD:R_0402_1005Metric, F.Cu at (96.5, 132.0)
- added R42: 270k, Resistor_SMD:R_0402_1005Metric, F.Cu at (128.6, 95.0)
- added R43: 100k, Resistor_SMD:R_0402_1005Metric, F.Cu at (128.6, 97.0)
- C1, C12, C26, C27, C4: footprint MySMD:SMD2012 -> Capacitor_SMD:C_0603_1608Metric
- C10: value NM -> 2.2p; footprint MySMD:SMD1005 -> Capacitor_SMD:C_0402_1005Metric
- C11, C14, C15, C17, C19, C2, C28, C29, C30, C31, C32, C33, C34, C37, C39, C41, C43, C44, C45, C8: footprint MySMD:SMD1005 -> Capacitor_SMD:C_0402_1005Metric
- C13: value 22n -> 0.1u; footprint MySMD:SMD1005 -> Capacitor_SMD:C_0402_1005Metric
- C16, C20: value 2.2p -> 1p; footprint MySMD:SMD1005 -> Capacitor_SMD:C_0402_1005Metric
- C18: footprint MySMD:SMD1608 -> Capacitor_SMD:C_0402_1005Metric
- C21: value 1u -> 0.1u; footprint MySMD:SMD1005 -> Capacitor_SMD:C_0402_1005Metric
- C25: value 4.7u 6.3V -> 4.7u 10V; footprint MySMD:SMD1608 -> Capacitor_SMD:C_0402_1005Metric
- C3: footprint MySMD:SMD2012 -> Capacitor_SMD:C_0805_2012Metric
- C35: value 4.7n 100V -> 15p; footprint MySMD:SMD1608 -> Capacitor_SMD:C_0402_1005Metric
- C36, C38: value 18p -> 10p; footprint MySMD:SMD1005 -> Capacitor_SMD:C_0402_1005Metric
- C42, C7: value 10u 6.3V -> 0.1u; footprint MySMD:SMD1608 -> Capacitor_SMD:C_0402_1005Metric
- C5: value 4.7p -> 6.8p; footprint MySMD:SMD1005 -> Capacitor_SMD:C_0402_1005Metric
- C6: value 120p -> 220p; footprint MySMD:SMD1005 -> Capacitor_SMD:C_0402_1005Metric
- C9: value NM -> 4.7p; footprint MySMD:SMD1005 -> Capacitor_SMD:C_0402_1005Metric
- CT1: value TZC3R100A110 3p-10p -> STC3MB10-T1
- CT2: value TZC3Z030A110R00 1.4p-3p -> STC3MA03-T1
- D1: value APT1608EC -> KT-0603R
- D2: value RB521S30T5G -> 1N5819WS; footprint MyDiode:SOD-523 -> Diode_SMD:D_SOD-323
- L2, L4: value LBR2012T202K -> LB2012T220K; footprint MySMD:SMD2012 -> Inductor_SMD:L_0805_2012Metric
- P2: value FCI_10118193-0001LF -> HRO TYPE-C-31-M-12; footprint MyJack:10118193-0001LF -> Connector_USB:USB_C_Receptacle_HRO_TYPE-C-31-M-12
- R1, R11, R36, R39, R40, R8: value 2.2k 5% -> 2.2k 1%; footprint MySMD:SMD1005 -> Resistor_SMD:R_0402_1005Metric
- R10, R13, R14, R15, R16, R2, R3, R31, R33, R34, R35, R37, R38, R4, R5, R6, R7, R9: footprint MySMD:SMD1005 -> Resistor_SMD:R_0402_1005Metric
- R12: value 10k 5% -> 2.2k 1%; footprint MySMD:SMD1005 -> Resistor_SMD:R_0402_1005Metric
- R17, R32: value 4.7k 5% -> 4.7k 1%; footprint MySMD:SMD1005 -> Resistor_SMD:R_0402_1005Metric
- R18: value 910 1% -> 2.2k 1%; footprint MySMD:SMD1005 -> Resistor_SMD:R_0402_1005Metric
- R19, R29: value 100 5% -> 100 1%; footprint MySMD:SMD1005 -> Resistor_SMD:R_0402_1005Metric
- R20, R22, R25, R26: value 4.7k -> 4.7k 1%; footprint MySMD:SMD1005 -> Resistor_SMD:R_0402_1005Metric
- R21: value 1k 1% -> 2.2k 1%; footprint MySMD:SMD1005 -> Resistor_SMD:R_0402_1005Metric
- R23: value 1M 5% -> 5.1k 1%; footprint MySMD:SMD1005 -> Resistor_SMD:R_0402_1005Metric
- R24: value 680 1% -> 470 1%; footprint MySMD:SMD1005 -> Resistor_SMD:R_0402_1005Metric
- R27, R28: value 1M 5% -> 1M 1%; footprint MySMD:SMD1005 -> Resistor_SMD:R_0402_1005Metric
- R30: value 0 -> 47; footprint MySMD:SMD1005 -> Resistor_SMD:R_0402_1005Metric
- U10, U14: footprint TO_SOT_Packages_SMD:SOT-23-6 -> Package_TO_SOT_SMD:SOT-23-6
- U11, U12: value LM385M3-1.2/NOPB -> LM385M3-1.2/TR; footprint TO_SOT_Packages_SMD:SOT-23 -> Package_TO_SOT_SMD:SOT-23-3
- U13: value AT24C02C-XHM-T -> FM24C02B-DN-T-G; footprint MyIC:TSSOP-8_4.4x3mm_Pitch0.65mm -> Package_DFN_QFN:TDFN-8-1EP_3x2mm_P0.5mm_EP1.4x1.4mm
- U2, U4: value CPC1017N -> CPC1017NTR
- U3: value AMS1117-3.3 -> MT3406; footprint MyIC:SOT-223 -> Package_TO_SOT_SMD:SOT-23-5
- U5: footprint MyIC:TSSOP-14_4.4x5mm_Pitch0.65mm -> Package_SO:TSSOP-14_4.4x5mm_P0.65mm
- U6: value LM2664 -> TI LM2664M6X/NOPB; footprint TO_SOT_Packages_SMD:SOT-23-6 -> Package_TO_SOT_SMD:SOT-23-6
- U7: footprint MyIC:TSSOP-16_4.4x5mm_Pitch0.65mm -> Package_SO:TSSOP-16_4.4x5mm_P0.65mm
- U8: value W25Q80BVSSIG -> ZD25WQ80CEIGR; footprint MyIC:SOIJ-8_5.3x5.3mm_Pitch1.27mm -> Package_SON:Winbond_USON-8-1EP_3x2mm_P0.5mm_EP0.2x1.6mm
- Y1: value ABLS-12.000MHZ-B4-T -> SCTF SX2B12.000F1010F30; footprint Crystals:Crystal_HC49-SD_SMD -> Crystal:Crystal_SMD_2520-4Pin_2.5x2.0mm
- moved C38 6.11 mm to (109.4, 112.7), turned to 180 degrees
- moved C36 5.94 mm to (107.3, 112.7), turned to 0 degrees
Connections:
- net LED0 renamed /LED_0
- net Net-(C10-Pad2) renamed /HIGH_VDIV
- net Net-(C5-Pad1) renamed /LOW_VDIV
- C11 pad 1: Net-(C11-Pad1) -> alt_3.3VD
- C13 pad 1: Net-(C11-Pad1) -> alt_3.3VD
- C14 pad 1: Net-(C11-Pad1) -> alt_3.3VD
- C21 pad 1: alt_VAA+ -> Net-(U14-VREF)
- C35 pad 1: Net-(C35-Pad1) -> alt_3.3VD
- C35 pad 2: GND -> Net-(U3-FB)
- C36 pad 1: GND -> Net-(U1B-XTAL2)
- C36 pad 2: Net-(C36-Pad2) -> GND
- C37 pad 1: Net-(C37-Pad1) -> Net-(U10-VBUS)
- C38 pad 1: GND -> Net-(U1B-XTAL1)
- C38 pad 2: Net-(C38-Pad2) -> GND
- C40 pad 2: Net-(C40-Pad2) -> Net-(U14-VREF)
- C7 pad 1: Net-(C11-Pad1) -> alt_3.3VD
- L5 pad 1: Net-(C37-Pad1) -> Net-(U10-VBUS)
- P2 pad S1: Net-(C35-Pad1) -> GND
- R23 pad 1: Net-(C35-Pad1) -> Net-(P2-CC1)
- R32 pad 2: Net-(C40-Pad2) -> Net-(U14-VREF)
- U1 pad A4: (no net) -> unconnected-(U1B-WAKEUP0-PadA4)
- U1 pad A5: (no net) -> unconnected-(U1B-RTCX1-PadA5)
- U1 pad A6: (no net) -> unconnected-(U1B-DBGEN-PadA6)
- U1 pad A8: (no net) -> unconnected-(U1D-P3_0-PadA8)
- U1 pad B1: Net-(C38-Pad2) -> Net-(U1B-XTAL1)
- U1 pad B3: (no net) -> unconnected-(U1B-ADC2-PadB3)
- U1 pad B5: (no net) -> unconnected-(U1B-RTCX2-PadB5)
- U1 pad C1: Net-(C36-Pad2) -> Net-(U1B-XTAL2)
- U1 pad C3: (no net) -> unconnected-(U1B-RTC_ALARM-PadC3)
- U1 pad C5: (no net) -> unconnected-(U1A-VBAT-PadC5)
- U1 pad C9: (no net) -> unconnected-(U1D-P6_11-PadC9)
- U1 pad D9: (no net) -> unconnected-(U1D-P2_4-PadD9)
- U1 pad E10: (no net) -> unconnected-(U1B-DM1-PadE10)
- U1 pad E4: Net-(C11-Pad1) -> alt_3.3VD
- U1 pad E5: Net-(C11-Pad1) -> alt_3.3VD
- U1 pad E8: (no net) -> unconnected-(U1D-P2_10-PadE8)
- U1 pad E9: (no net) -> unconnected-(U1B-DP1-PadE9)
- U1 pad F1: (no net) -> unconnected-(U1C-USB0_ID-PadF1)
- U1 pad F4: Net-(C11-Pad1) -> alt_3.3VD
- U1 pad F5: (no net) -> unconnected-(U1D-P2_2-PadF5)
- U1 pad F6: (no net) -> unconnected-(U1D-P6_4-PadF6)
- U1 pad F7: (no net) -> unconnected-(U1D-P3_1-PadF7)
- U1 pad F8: (no net) -> unconnected-(U1D-P6_9-PadF8)
- U1 pad F9: (no net) -> unconnected-(U1D-P6_5-PadF9)
- U1 pad G1: (no net) -> unconnected-(U1D-P0_1-PadG1)
- U1 pad G10: (no net) -> unconnected-(U1D-P2_0-PadG10)
- U1 pad G2: (no net) -> unconnected-(U1D-P0_0-PadG2)
- U1 pad G4: (no net) -> unconnected-(U1D-P1_7-PadG4)
- U1 pad G5: (no net) -> unconnected-(U1D-P6_1-PadG5)
- U1 pad G6: (no net) -> unconnected-(U1D-P3_2-PadG6)
- U1 pad G7: (no net) -> unconnected-(U1D-P2_1-PadG7)
- U1 pad H1: (no net) -> unconnected-(U1D-P1_0-PadH1)
- U1 pad H10: (no net) -> unconnected-(U1D-P1_17-PadH10)
- U1 pad H4: (no net) -> unconnected-(U1D-PF_4-PadH4)
- U1 pad H5: (no net) -> unconnected-(U1D-P1_8-PadH5)
- U1 pad H6: (no net) -> unconnected-(U1D-P1_10-PadH6)
- U1 pad H7: (no net) -> unconnected-(U1D-P6_0-PadH7)
- U1 pad H8: (no net) -> unconnected-(U1D-P1_13-PadH8)
- U1 pad H9: (no net) -> unconnected-(U1D-P1_16-PadH9)
- U1 pad J1: (no net) -> unconnected-(U1D-P1_3-PadJ1)
- U1 pad J10: (no net) -> unconnected-(U1D-P1_18-PadJ10)
- U1 pad J2: (no net) -> unconnected-(U1D-P1_4-PadJ2)
- U1 pad J4: (no net) -> unconnected-(U1D-P1_5-PadJ4)
- U1 pad J5: (no net) -> unconnected-(U1D-P1_9-PadJ5)
- U1 pad J7: (no net) -> unconnected-(U1D-P1_11-PadJ7)
- U1 pad J8: (no net) -> unconnected-(U1D-P1_14-PadJ8)
- U1 pad J9: (no net) -> unconnected-(U1D-P6_2-PadJ9)
- U1 pad K2: (no net) -> BOOT0
- U1 pad K3: (no net) -> unconnected-(U1B-CLK0-PadK3)
- U1 pad K6: (no net) -> unconnected-(U1B-CLK2-PadK6)
- U1 pad K7: (no net) -> unconnected-(U1D-P1_12-PadK7)
- U1 pad K8: (no net) -> unconnected-(U1D-P1_15-PadK8)
- U1 pad K9: (no net) -> unconnected-(U1D-P1_19-PadK9)
- U10 pad 5: Net-(C37-Pad1) -> Net-(U10-VBUS)
- U11 pad 3: (no net) -> unconnected-(U11-NC-Pad3)
- U12 pad 3: (no net) -> unconnected-(U12-NC-Pad3)
- U14 pad 6: Net-(C40-Pad2) -> Net-(U14-VREF)
- U3 pad 1: GND -> VBUS
- U3 pad 2: alt_3.3VD -> GND
- U3 pad 3: VBUS -> Net-(U3-SW)
- U3 pad 4: (no net) -> VBUS
- U7 pad 11: (no net) -> unconnected-(U7-X3-Pad11)
- U7 pad 4: (no net) -> unconnected-(U7-Y3-Pad4)
- Y1 pad 1: Net-(C36-Pad2) -> Net-(U1B-XTAL2)
- Y1 pad 2: Net-(C38-Pad2) -> Net-(U1B-XTAL1)
Routing:
- net (no net): track 0.00 -> 80.7 mm, vias 0 -> 7
- net Net-(C37-Pad1): track 34.7 -> 0.00 mm, vias 7 -> 0
- net Net-(C11-Pad1): track 29.6 -> 0.00 mm, vias 8 -> 0
- net Net-(C36-Pad2): track 27.6 -> 0.00 mm
- net Net-(C35-Pad1): track 16.3 -> 0.00 mm
- net Net-(C38-Pad2): track 14.7 -> 0.00 mm
- net Net-(U1B-XTAL1): track 0.00 -> 9.77 mm
- net GND: track 94.9 -> 85.2 mm, vias 69 -> 63
- net Net-(U1B-XTAL2): track 0.00 -> 9.25 mm
- net SPIFI_CS: track 21.8 -> 15.9 mm
- net Net-(U14-VREF): track 0.00 -> 4.40 mm
- net Net-(C40-Pad2): track 4.40 -> 0.00 mm
- net I2C_SDA: track 29.7 -> 28.3 mm, vias 4 -> 3
- net alt_3.3VD: track 220.6 -> 219.4 mm, vias 15 -> 22
- net I2C_SCL: track 30.0 -> 28.9 mm, vias 3 -> 2
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- added copper zone on In2.Cu, net GND
- removed copper zone on In2_GND.Cu, net GND
Other:
- net class Default removed
- net class Power removed
