File: USB_Oscilloscope.kicad_sch (KiCad schematic)
At the start: 116 parts, among them J1 Needle, P1 USB_BOOT, P2 HRO TYPE-C-31-M-12, P3 JTAG, SW1 MSK12C02, U1 LPC4370FET100, U10 USBLC6-2SC6, U11 LM385M3-1.2/TR, U12 LM385M3-1.2/TR, U13 FM24C02B-DN-T-G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

Commit message: プロジェクト名変更
Parts:
- removed D3: BAS16VY, Package_TO_SOT_SMD:SOT-363_SC-70-6, symbol #ps_symbol:BAS16V
- removed P1: USB_BOOT, Connector_PinHeader_1.27mm:PinHeader_1x02_P1.27mm_Vertical, symbol Connector_Generic:Conn_01x02
- removed P3: JTAG, #ps_foot:PIN_HEADER_7_1.27pitch, symbol Connector_Generic:Conn_01x07
- removed R11, R39, R40: 2.2k 1%, Resistor_SMD:R_0402_1005Metric, symbol Device:R
- removed R25: 4.7k 1%, Resistor_SMD:R_0402_1005Metric, symbol Device:R
- removed R29: 100 1%, Resistor_SMD:R_0402_1005Metric, symbol Device:R
- removed W1: ISP, TestPoint:TestPoint_Pad_1.0x1.0mm, symbol Connector:TestPoint
- added J1: POGO_PROG, #ps_foot:PIN_HEADER_P1.27x4, symbol Connector_Generic:Conn_01x04
- added J3: DEBUG, #ps_foot:JST_SH_SM06B-SRSS-TB_1x06-1MP_P1.00mm_Horizontal, symbol #ps_symbol:SWD_AND_UART_6PIN
- added U15: LM385M3-1.2/TR, Package_TO_SOT_SMD:SOT-23-3, symbol #ps_symbol:LM385M3
- C10: LCSC (none) -> C1559
- C16, C20: LCSC (none) -> C1550
- C22: footprint Capacitor_SMD:C_0402_1005Metric -> Capacitor_SMD:C_0603_1608Metric; LCSC (none) -> C3890240
- C29: LCSC (none) -> C1565
- C32, C9: LCSC (none) -> C1569
- C36, C38: value 10p -> 18p; LCSC C32949 -> (none)
- C5: LCSC (none) -> C1576
- PAD1: renamed from J1; value Needle -> TIP WIRE; footprint (none) -> #ps_foot:TIP_WIRE; now left out of the parts list
- R10, R9: LCSC (none) -> C25771
- R15: LCSC (none) -> C25908
- R16: LCSC (none) -> C122547
- R2: LCSC (none) -> C133039
- R24: LCSC (none) -> C25117
- R27: footprint Resistor_SMD:R_0603_1608Metric -> Resistor_SMD:R_0805_2012Metric; LCSC (none) -> C17668
- R28: footprint Resistor_SMD:R_0603_1608Metric -> Resistor_SMD:R_0805_2012Metric; LCSC (none) -> C17674
- R3: LCSC (none) -> C25800
- R30: LCSC (none) -> C25118
- R34: LCSC (none) -> C25924
- R4: LCSC (none) -> C477601
- R42: LCSC (none) -> C25770
- R43: LCSC (none) -> C25741
- R5: LCSC (none) -> C43676
- TP3: now left out of the parts list
- W3, W5: footprint TestPoint:TestPoint_Pad_1.0x1.0mm -> TestPoint:TestPoint_Pad_D1.0mm; now left out of the parts list
- Y1: value SCTF SX2B12.000F1010F30 -> 7E12000E20UCG; LCSC C7301971 -> C252259
Connections:
- net BOOT1 is gone; now on net GND: U1.K1 (P1_2_BOOT)
- net BOOT2 is gone; now on net GND: U1.C6 (P2_8_BOOT)
- net BOOT3 is gone; now on net GND: U1.B10 (P2_9_BOOT)
- net GND: now also J1.2 (Pin_2), J3.3 (GND), U15.2
- net LOW_VDIV: now also U4.3 (INOUT2); no longer U4.4 (INOUT1)
- net VDD: now also U1.E3 (USB0_VBUS), J1.4 (Pin_4), J3.1 (V_TARGET)
- net at C22.1, C3.1, CT3.2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: now also SW1.1 (A); no longer SW1.3 (C)
- net at U5.3 (+IN): now also U4.4 (INOUT1); no longer U4.3 (INOUT2)
- net at D2.1 (K), R24.2, U5.5 (+IN): now also U15.1
- net RESET: now reaches R26.2, TP3.1, U1.B6 (RESET#)
- net RESET: now also J3.5 (NRST)
- net at C22.2, CT3.1, R27.1: now also PAD1.1 (Pin_1), SW1.2 (B); no longer SW1.1 (A)
- net BOOT0: no longer names the net of U1.K2 (P1_1_BOOT)
- net BOOT_ISP: no longer names the net of U1.C10 (P2_7_ISP)
- net JTAG_RESET: no longer names the net of U1.B4 (TRST#)
- net JTAG_TCK renamed SWCLK
- net SWCLK: now also J1.3 (Pin_3), J3.2 (SWCLK)
- net JTAG_TDI: no longer names the net of U1.G3 (JTDI)
- net JTAG_TDO renamed SWO
- net SWO: now also J3.6 (SWO)
- net JTAG_TMS renamed SWDIO
- net SWDIO: now also J1.1 (Pin_1), J3.4 (SWDIO)
- net OP_SW renamed OP_LOW_SW
- no-connect marks 55 -> 60
Other:
- note added: "ADC protection voltage clipper -0.2V ~ +1.2V"
- note removed: "ADC protection diode -0.2V - 1.8V"
- note removed: "BOOT select resistors (LPC4370 pins are default weak pull up)"
- note removed: "Photo MOS Switch"
- company: PulseLime -> LimePulse
- title: DroidOscillo schematic -> Open Pen Type Oscilloscope
- moved on the sheet: C11, C13, C14, C17, C19, C21, C22, C30, C34, C36, C38, C41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

Commit message: ペン型オシロに変更
Parts:
- removed P2: HRO TYPE-C-31-M-12, Connector_USB:USB_C_Receptacle_HRO_TYPE-C-31-M-12, symbol Connector:USB_C_Receptacle_USB2.0_16P
- removed R23, R41: 5.1k 1%, Resistor_SMD:R_0402_1005Metric, symbol Device:R
- removed W3: ADC1, TestPoint:TestPoint_Pad_D1.0mm, symbol Connector:TestPoint
- added C23, C24, C46: 0.1u, Capacitor_SMD:C_0402_1005Metric, symbol Device:C
- added C37, C40: 1u, Capacitor_SMD:C_0402_1005Metric, symbol Device:C
- added J1: Solder pads 1x04, #ps_foot:01x04_wire_pads_Pitch2.0, symbol Connector_Generic:Conn_01x04
- added PAD2: SHIELD TUBE, #ps_foot:pipe-out5.0_in4.0_len40.0, symbol Connector_Generic:Conn_01x01
- CT1: renamed from CT3; footprint #ps_foot:MURATA_TZC3 -> #ps_foot:SHEWA STC03M
- CT2: renamed from CT1; footprint #ps_foot:MURATA_TZC3 -> #ps_foot:SHEWA STC03M
- CT3: renamed from CT2; footprint #ps_foot:MURATA_TZC3 -> #ps_foot:SHEWA STC03M
- J3: LCSC (none) -> C7430448; now in the parts list
- R42: value 270k -> 100k 1%; LCSC C25770 -> C25741
- R43: value 100k -> 22k 1%; LCSC C25741 -> C25768
- SW1: value MSK12C02 -> MSS12C02LS-BB2.0; footprint #ps_foot:MSK12C02 -> #ps_foot:MSS12C02LS-BB2.0; LCSC C431540 -> C3008585
- TP3: footprint TestPoint:TestPoint_Pad_1.0x1.0mm -> TestPoint:TestPoint_Pad_D1.0mm
- U13: footprint Package_DFN_QFN:TDFN-8-1EP_3x2mm_P0.5mm_EP1.4x1.4mm -> #ps_foot:TDFN-8-1EP_3x2mm_P0.5mm_EP1.4x1.4mm
- U7: value 74HC4052PW -> 74HC4052PW,118
- renumbered J1 to J2, W5 to TP2
Connections:
- net GND: now also C23.2, C24.1, C37.2, C40.1, C46.2, J1.4 (Pin_4), PAD2.1 (Pin_1); no longer SW1.S1, SW1.S2, SW1.S3, SW1.S4
- net USB_D+: now also U10.1 (IO1), U10.6 (IO1), J1.3 (Pin_3); no longer U10.3 (IO2), U10.4 (IO2)
- net USB_D-: now also U10.3 (IO2), U10.4 (IO2), J1.2 (Pin_2); no longer U10.1 (IO1), U10.6 (IO1)
- net USB_VBUS: now also J1.1 (Pin_1)
- net VDD: now also C46.1
- net alt_VAA+: now also C23.1, C37.1
- net alt_VAA-: now also C24.2, C40.2
- net H_OP_OUT: now reaches C16.1, C29.2, C31.2, R14.2, R15.2, R9.2, U7.1 (Y0), U9.7 (Ch0)
- net H_OP_OUT: now also U5.8 (OUT); no longer U5.14 (OUT)
- net L_OP_OUT: now reaches C20.2, C28.1, C32.1, R10.1, R13.1, R16.1, U7.12 (X0), U9.6 (Ch1)
- net L_OP_OUT: now also U5.7 (OUT); no longer U5.1 (OUT)
- net L_OP-: now reaches C20.1, R10.2, R6.1, U7.13 (X)
- net L_OP-: now also U5.6 (-IN); no longer U5.2 (-IN)
- net H_OP-: now reaches C16.2, R7.1, R9.1, U7.3 (Y)
- net H_OP-: now also U5.9 (-IN); no longer U5.13 (-IN)
- net DIV_IN_40V: now reaches C10.1, C3.2, C9.1, R2.2, R4.1, U2.4 (INOUT1)
- net DIV_IN_40V: now also CT2.2, CT3.2; no longer CT2.1, CT3.1
- net DCC_IN_40V: now reaches C22.1, C3.1, CT1.2, R28.2, U2.3 (INOUT2)
- net DCC_IN_40V: now also SW1.2 (B); no longer SW1.1 (A)
- net L_OP+: now reaches U4.4 (INOUT1)
- net L_OP+: now also U5.5 (+IN); no longer U5.3 (+IN)
- net OP_CLP-: now reaches R18.1, R21.2
- net OP_CLP-: now also U5.2 (-IN); no longer U5.9 (-IN)
- net at R21.1, R24.1: now also U5.1 (OUT); no longer U5.8 (OUT)
- net OP_VF+: now reaches D2.1 (K), R24.2, U15.1
- net OP_VF+: now also U5.12 (+IN); no longer U5.5 (+IN)
- net OP_CLP+: now reaches C33.1, R17.2
- net OP_CLP+: now also U5.3 (+IN); no longer U5.10 (+IN)
- net TIP_400V: now reaches C22.2, CT1.1, PAD1.1 (Pin_1), R27.1
- net TIP_400V: now also SW1.1 (A); no longer SW1.2 (B)
- net HIGH_VDIV renamed H_DIV
- net H_DIV: now also CT3.1, U5.10 (+IN); no longer CT3.2, U5.12 (+IN)
- net LOW_VDIV renamed L_DIV
- net L_DIV: now also CT2.1; no longer CT2.2
- new net OP_VF-: R30.1, U5.13 (-IN), U5.14 (OUT)
- no-connect marks 60 -> 63
Other:
- note added: "HIGH VOLTAGE INPUT ATTENUETION 1.8% Max40Vp-p (1x)"
- note removed: "1M_IMP"
- note removed: "HIGH VOLTAGE INPUT ATTENUETION 1.8%"
- moved on the sheet: C35, R18, U5A, U5B, U5C, U5D, U5E
